File: blacker-cannon-cards/blacker-cannon-cards.kicad_pcb (KiCad board)
At the start: 2 copper layers, 85 x 55 mm, 7 parts

Commit message: Regenerate Gerbers for JLC production
Other:
- board text added: "JLCJLCJLCJLC"
Changed lines of the file:
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@@
   (general
     (thickness 1.6)
-    (drawings 14)
+    (drawings 15)
     (tracks 0)
     (zones 0)
@@
       (xy 13.779922 -9.004775) (xy 18.282034 -4.502332)) (layer F.Mask) (width 0.01))
   )
+  (gr_text JLCJLCJLCJLC (at 59 103.5) (layer B.SilkS)
+    (effects (font (size 0.83 0.83) (thickness 0.2)) (justify mirror))
+  )
   (gr_arc (start 130 100) (end 130 105) (angle -90) (layer Edge.Cuts) (width 0.05))
